File: pcb/quantumpad.kicad_pcb (KiCad board)
At the start: 2 copper layers, 100 x 100 mm, 25 parts, among them SW2 RotaryEncoder_Switch, U17 MOUDLE-SEEEDUINO-XIAO

Commit message: Added BOM and updated images/PCB/gerber
Connections:
- U17 pad 12: unconnected-(U17-3V3-Pad12) -> Net-(D11-VCC)
- U17 pad 14: Net-(D11-VCC) -> unconnected-(U17-5V-Pad14)
Routing:
- net Net-(D11-VCC): track 57.0 -> 56.2 mm
Changed lines of the file:
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@@
 			(outputformat 1)
 			(mirror no)
-			(drillshape 1)
+			(drillshape 0)
 			(scaleselection 1)
-			(outputdirectory "")
+			(outputdirectory "quantumpad-gerber")
 		)
 	)
@@
 	(net 20 "/COL2")
 	(net 21 "/COL3")
-	(net 22 "unconnected-(U17-3V3-Pad12)")
+	(net 22 "unconnected-(U17-5V-Pad14)")
 	(net 23 "Net-(U17-PA11_A3_D3)")
 	(footprint "Diode_THT:D_DO-35_SOD27_P7.62mm_Horizontal"
@@
 			(layers "*.Cu" "*.Mask")
 			(remove_unused_layers no)
-			(net 22 "unconnected-(U17-3V3-Pad12)")
+			(net 4 "Net-(D11-VCC)")
 			(pinfunction "3V3")
 			(pintype "passive")
@@
 			(layers "F.Cu" "F.Mask" "F.Paste")
 			(roundrect_rratio 0.25)
-			(net 22 "unconnected-(U17-3V3-Pad12)")
+			(net 4 "Net-(D11-VCC)")
 			(pinfunction "3V3")
 			(pintype "passive")
@@
 			(layers "*.Cu" "*.Mask")
 			(remove_unused_layers no)
-			(net 4 "Net-(D11-VCC)")
+			(net 22 "unconnected-(U17-5V-Pad14)")
 			(pinfunction "5V")
 			(pintype "passive")
@@
 			(layers "F.Cu" "F.Mask" "F.Paste")
 			(roundrect_rratio 0.25)
-			(net 4 "Net-(D11-VCC)")
+			(net 22 "unconnected-(U17-5V-Pad14)")
 			(pinfunction "5V")
 			(pintype "passive")
@@
 		(net 3)
 	)
-	(segment
-		(start 185.963 26.537)
-		(end 187.6175 26.537)
-		(width 0.2)
-		(layer "F.Cu")
-		(net 4)
-	)
-	(segment
-		(start 182.5 30)
-		(end 185.963 26.537)
-		(width 0.2)
-		(layer "F.Cu")
-		(net 4)
-	)
 	(via
 		(at 182.5 30)
@@
 	)
 	(segment
+		(start 184.117 31.617)
+		(end 187.6175 31.617)
+		(width 0.2)
+		(layer "B.Cu")
+		(net 4)
+	)
+	(segment
+		(start 182.5 30)
+		(end 184.117 31.617)
+		(width 0.2)
+		(layer "B.Cu")
+		(net 4)
+	)
+	(segment
 		(start 95.44 72.35)
 		(end 95.44 68.8)
@@
 		(width 0.2)
 		(layer "B.Cu")
-		(net 13)
-	)
-	(segment
-		(start 188.6175 53.737)
-		(end 188.6175 53.6175)
-		(width 0.2)
-		(layer "B.Cu")
